File: AnalogOscillator.kicad_sch (KiCad schematic)
At the start: 59 parts, among them J2 031-71052, J3 031-71052, J4 031-71052, J5 031-71052, J6 5442183, J7 031-71052, J8 031-71052, P2 RK09D113F25C0B504, P3 RK09D113F25C0B504, U1 OPA134PA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

Commit message: Updated connectors and SMD components
Parts:
- removed J4, J5, J8: 031-71052, 031-71052:03171052, symbol 031-71052:031-71052
- removed R12: 1k, Resistor_THT:R_Axial_DIN0207_L6.3mm_D2.5mm_P7.62mm_Horizontal, symbol Device:R_US
- removed R13, R14, R15, R16: 10k, Resistor_THT:R_Axial_DIN0207_L6.3mm_D2.5mm_P7.62mm_Horizontal, symbol Device:R_US
- removed R8: 100k, Resistor_THT:R_Axial_DIN0207_L6.3mm_D2.5mm_P7.62mm_Horizontal, symbol Device:R_US
- added J1, J4: B4B-XH-A, B4B_XH_A:JST_B4B-XH-A, symbol B4B-XH-A:B4B-XH-A
- added R1: ERA-3AEB102V, ERA-3AEB:ERA3AEB101V, symbol ERA-3AEB102V:ERA-3AEB102V
- added R2, R3, R5, R7, R8: ERA-3AEB103V, ERA-3AEB:ERA3AEB101V, symbol ERA-3AEB103V:ERA-3AEB103V
- added R6, R9: ERA-3AEB104V, ERA-3AEB:ERA3AEB101V, symbol ERA-3AEB104V:ERA-3AEB104V
- C1, C2: value 1uF -> ECW-FD2W105J
Connections:
- net -V: now also U12.6 (OUTPUT), R8.2
- net -x: now also R3.2
- net GND: now also J1.4, J4.4
- net Sum: now also R6.2
- net V: now also R1.1, R7.1
- net VR1: now also U5.2 (IN-), U5.6 (OUTPUT), R9.1
- net VR2: now also U4.2 (IN-), U4.6 (OUTPUT), R5.1
- net VR4: now also R6.1
- net x: now also R2.1
- net V_out: now reaches U8.2 (IN-), U8.6 (OUTPUT)
- net V_out: now also J1.2
- net at C2.1, U2.2 (IN-): now also R1.2
- net at U12.2 (IN-): now also R7.2, R8.1
- net X_out: now reaches U9.2 (IN-), U9.6 (OUTPUT)
- net X_out: now also J1.1
- net at U3.2 (IN-): now also R2.2, R3.1
- net at U13.3 (IN+): now also J4.3
- new net S_out: J1.3, R5.2, R9.2
