File: AnalogOscillator.kicad_sch (KiCad schematic)
At the start: 60 parts, among them J1 B4B-XH-A, J2 031-71052, J3 031-71052, J4 B4B-XH-A, J6 5442183, J7 031-71052, P2 RK09D113F25C0B504, P3 RK09D113F25C0B504, U1 OPA134PA, U11 OPA134PA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

Commit message: "{""Full Name"":""James"",""Date of Birth"":""23/04/1985"",""Health Conditions"":""Alzheimer's, Arthritis, Dementia, Cognitive decline"",""Medications"":""Aspirin: ; Lecanemab: ; donanemab: "",""Daily Routine Summary"":""Wake up, take a walk, go swimming, sleep, read a book, have lunch, take a nap, walk the dog, watch tv, read the news, have dinner, journal, sleep""}","{""Emotional Triggers"":""Seeing graveyards"",""Comforting Methods"":""Looking at a picture of my wife"",""Medical History"":""Tends to get spasms and sudden depression""}","{""Home Address"":""123, Sardar Patel Road, Chennai"",""Preferred Hospital"":""Anna Nagar Hospital"",""Voice Prompt Script"":""""}","Kusuma (child): 9438394982 - She works in another city; Rodrigues (other): 39843984 - Neighbor next door, regular visitor","{""Routine Events"":""{\""01:00\"":\""Take medicine\"",\""03:00\"":\""Eat lunch\"",\""04:00\"":\""Take a walk\"",\""05:00\"":\""Sleep\"",\""11:00\"":\""Wake up\"",\""13:00\"":\""Have food\"",\""15:00\"":\""Read the news\"",\""16:00\"":\""Cook food for myself\"",\""19:00\"":\""Visit the local restaurant\"",\""21:00\"":\""Take second nap\""}"",""Memory Description"":""The time i saw a monkey and realised my passion to be a zookeeper"",""Safety Notes"":""Stay away from orangutans"",""Uploaded Image"":""No Image Uploaded""}",Glasses - In the kitchen; Tablets - Under the bed; Car - The driveway; Spoons - Kitchen cabinet%
Parts:
- removed R5: ERA-3AEB103V, ERA-3AEB:ERA3AEB101V, symbol ERA-3AEB103V:ERA-3AEB103V
- removed R9: ERA-3AEB104V, ERA-3AEB:ERA3AEB101V, symbol ERA-3AEB104V:ERA-3AEB104V
- added J5: B4B-XH-A, B4B_XH_A:JST_B4B-XH-A, symbol B4B-XH-A:B4B-XH-A
- added R10: ERA-3AEB104V, ERA-3AEB:ERA3AEB101V, symbol ERA-3AEB104V:ERA-3AEB104V
- added R11: ERA-3AEB103V, ERA-3AEB:ERA3AEB101V, symbol ERA-3AEB103V:ERA-3AEB103V
- added S5, S6: LC1258EENP, LC1258EENP:SW_LC1258EENP, symbol LC1258EENP:LC1258EENP
Connections:
- net +15V: now also J5.1
- net -15V: now also J5.2
- net GND: now also J5.4
- net Sum: now also R6.1; no longer C1.1, R6.2, U1.2 (IN-)
- net VR1: now also R10.1
- net VR2: now also R11.1
- net VR4: no longer R6.1
- new net: C1.1, R6.2, S5.1, S6.1, U1.2 (IN-)
- new net: R10.2, S5.2
- new net: R11.2, S6.2
Other:
- note added: "Signal Generator"
- note removed: "Summer"
- title: (none) -> Primary Oscillation Engine
- moved on the sheet: C1, C10, C11, C12, C13, C14, C15, C16, C17, C18, C19, C2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
