File: _autosave-AnalogOscillator.kicad_sch (KiCad schematic)
At the start: 60 parts, among them J1 B4B-XH-A, J2 031-71052, J3 031-71052, J4 B4B-XH-A, J6 5442183, J7 031-71052, P2 RK09D113F25C0B504, P3 RK09D113F25C0B504, U1 OPA134PA, U11 OPA134PA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

Commit message: Updated
Other:
- note added: "Signal Generator"
- title: (none) -> Primary Oscillation Engine
- moved on the sheet: C1, C10, C11, C12, C13, C14, C15, C16, C17, C18, C19, C2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
