File: AnalogOscillator.kicad_pcb (KiCad board)
At the start: 2 copper layers, 200.5 x 120.5 mm, 59 parts, among them J2 031-71052, J3 031-71052, J4 031-71052, J5 031-71052, J6 5442183, J7 031-71052, J8 031-71052, P2 RK09D113F25C0B504, P3 RK09D113F25C0B504, U1 OPA134PA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

Commit message: Updated connectors and SMD components
Parts:
- removed J5, J8: 031-71052, 031-71052:03171052
- removed R12: 1k, Resistor_THT:R_Axial_DIN0207_L6.3mm_D2.5mm_P7.62mm_Horizontal
- removed R13, R14, R15, R16: 10k, Resistor_THT:R_Axial_DIN0207_L6.3mm_D2.5mm_P7.62mm_Horizontal
- added J1: B4B-XH-A, B4B_XH_A:JST_B4B-XH-A, F.Cu at (45.0, 45.0)
- added R1: ERA-3AEB102V, ERA-3AEB:ERA3AEB101V, F.Cu at (99.3, 45.0)
- added R2: ERA-3AEB103V, ERA-3AEB:ERA3AEB101V, F.Cu at (124.8, 46.0)
- added R3: ERA-3AEB103V, ERA-3AEB:ERA3AEB101V, F.Cu at (158.3, 45.0)
- added R5: ERA-3AEB103V, ERA-3AEB:ERA3AEB101V, F.Cu at (223.3, 73.0)
- added R6: ERA-3AEB104V, ERA-3AEB:ERA3AEB101V, F.Cu at (55.7, 44.0)
- added R7: ERA-3AEB103V, ERA-3AEB:ERA3AEB101V, F.Cu at (168.8, 45.0)
- added R9: ERA-3AEB104V, ERA-3AEB:ERA3AEB101V, F.Cu at (223.8, 81.0)
- C1, C2: value 1uF -> ECW-FD2W105J
- J4: value 031-71052 -> B4B-XH-A; footprint 031-71052:03171052 -> B4B_XH_A:JST_B4B-XH-A
- R8: value 100k -> ERA-3AEB103V; footprint Resistor_THT:R_Axial_DIN0207_L6.3mm_D2.5mm_P7.62mm_Horizontal -> ERA-3AEB:ERA3AEB101V
- moved R8 70.0 mm to (193.0, 45.0)
- moved J4 17.1 mm to (235.5, 76.8)
- moved J7 0.71 mm to (166.9, 133.4)
Connections:
- net Net-(J5-SIGNAL) renamed X_out
- net Net-(U4-IN-) renamed VR2
- net Net-(U5-IN-) renamed VR1
- J4 pad 1: Net-(J4-SIGNAL) -> unconnected-(J4-Pad1)
- J4 pad 2: GND -> unconnected-(J4-Pad2)
- R8 pad 1: Sum -> Net-(U12-IN-)
- R8 pad 2: VR4 -> -V
- U12 pad 6: Net-(U12-OUTPUT) -> -V
- U13 pad 3: Net-(J8-SIGNAL) -> Net-(U13-IN+)
- U8 pad 2: Net-(J4-SIGNAL) -> V_out
- U8 pad 6: Net-(J4-SIGNAL) -> V_out
Routing:
- net +15V: track 571.3 -> 0.00 mm, vias 1 -> 0
- net -15V: track 536.5 -> 0.00 mm
- net V: track 269.2 -> 0.00 mm, vias 1 -> 0
- net x: track 220.4 -> 0.00 mm, vias 2 -> 0
- net Sum: track 160.7 -> 0.00 mm, vias 1 -> 0
- net -x: track 97.4 -> 0.00 mm, vias 1 -> 0
- net Net-(U2-IN-): track 82.4 -> 0.00 mm
- net Net-(U3-IN-): track 45.4 -> 0.00 mm
- net Net-(U12-IN-): track 40.7 -> 0.00 mm
- net Net-(S3-Pad1): track 34.7 -> 0.00 mm
- net Net-(J8-SIGNAL): track 30.1 -> 0.00 mm
- net Net-(S1-Pad2): track 30.0 -> 0.00 mm
- net Net-(J4-SIGNAL): track 29.9 -> 0.00 mm
- net Net-(P3-WIPER): track 28.4 -> 0.00 mm
- net Net-(P2-WIPER): track 28.1 -> 0.00 mm
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- removed copper zone on F.Cu, net GND

Commit message: Updated
Parts:
- moved C21 5.39 mm to (178.0, 84.0)
- moved C17 4.03 mm to (63.0, 126.0)
- moved C8 3.62 mm to (104.5, 60.5)
- moved C19 2.50 mm to (113.5, 127.5)
- moved J1 1.99 mm to (47.0, 44.8)
- moved R6 1.04 mm to (56.0, 45.0)
Routing:
- net -15V: track 0.00 -> 570.4 mm, vias 0 -> 1
- net V: track 0.00 -> 277.5 mm, vias 0 -> 2
- net X_out: track 0.00 -> 225.3 mm, vias 0 -> 1
- net S_out: track 0.00 -> 204.1 mm, vias 0 -> 1
- net x: track 0.00 -> 204.0 mm
- net VR4: track 0.00 -> 183.0 mm, vias 0 -> 2
- net V_out: track 0.00 -> 177.9 mm, vias 0 -> 1
- net Net-(U13-IN+): track 0.00 -> 174.8 mm, vias 0 -> 1
- net -V: track 0.00 -> 173.2 mm, vias 0 -> 1
- net VR1: track 0.00 -> 156.3 mm
- net VR2: track 0.00 -> 106.7 mm
- net -x: track 0.00 -> 96.7 mm, vias 0 -> 1
- net Net-(U2-IN-): track 0.00 -> 83.0 mm
- net Sum: track 0.00 -> 71.9 mm
- net Net-(U3-IN-): track 0.00 -> 58.6 mm
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- added copper zone on F.Cu, net +15V
- added copper zone on B.Cu, net GND

Commit message: "{""Full Name"":""James"",""Date of Birth"":""23/04/1985"",""Health Conditions"":""Alzheimer's, Arthritis, Dementia, Cognitive decline"",""Medications"":""Aspirin: ; Lecanemab: ; donanemab: "",""Daily Routine Summary"":""Wake up, take a walk, go swimming, sleep, read a book, have lunch, take a nap, walk the dog, watch tv, read the news, have dinner, journal, sleep""}","{""Emotional Triggers"":""Seeing graveyards"",""Comforting Methods"":""Looking at a picture of my wife"",""Medical History"":""Tends to get spasms and sudden depression""}","{""Home Address"":""123, Sardar Patel Road, Chennai"",""Preferred Hospital"":""Anna Nagar Hospital"",""Voice Prompt Script"":""""}","Kusuma (child): 9438394982 - She works in another city; Rodrigues (other): 39843984 - Neighbor next door, regular visitor","{""Routine Events"":""{\""01:00\"":\""Take medicine\"",\""03:00\"":\""Eat lunch\"",\""04:00\"":\""Take a walk\"",\""05:00\"":\""Sleep\"",\""11:00\"":\""Wake up\"",\""13:00\"":\""Have food\"",\""15:00\"":\""Read the news\"",\""16:00\"":\""Cook food for myself\"",\""19:00\"":\""Visit the local restaurant\"",\""21:00\"":\""Take second nap\""}"",""Memory Description"":""The time i saw a monkey and realised my passion to be a zookeeper"",""Safety Notes"":""Stay away from orangutans"",""Uploaded Image"":""No Image Uploaded""}",Glasses - In the kitchen; Tablets - Under the bed; Car - The driveway; Spoons - Kitchen cabinet%
Parts:
- removed R5: ERA-3AEB103V, ERA-3AEB:ERA3AEB101V
- removed R9: ERA-3AEB104V, ERA-3AEB:ERA3AEB101V
- added J5: B4B-XH-A, B4B_XH_A:JST_B4B-XH-A, F.Cu at (184.5, 94.8)
- added R10: ERA-3AEB104V, ERA-3AEB:ERA3AEB101V, F.Cu at (48.8, 40.0)
- added R11: ERA-3AEB103V, ERA-3AEB:ERA3AEB101V, F.Cu at (48.5, 55.5)
- added S5: LC1258EENP, LC1258EENP:SW_LC1258EENP, F.Cu at (58.0, 32.5)
- added S6: LC1258EENP, LC1258EENP:SW_LC1258EENP, F.Cu at (58.3, 61.2)
- moved C33 53.5 mm to (182.5, 116.0), turned to -90 degrees
- moved J4 51.0 mm to (184.5, 75.8)
- moved C23 40.6 mm to (148.0, 104.0)
- moved C24 40.6 mm to (169.0, 103.5)
- moved U9 40.6 mm to (162.1, 102.6)
- moved J6 40.2 mm to (183.0, 123.5), turned to -90 degrees
- moved C29 32.6 mm to (171.5, 36.5)
- moved C30 32.6 mm to (172.0, 58.0)
- moved U12 32.6 mm to (172.9, 51.6)
- moved C22 32.5 mm to (172.5, 82.5)
- moved U8 32.5 mm to (165.6, 81.0)
- moved C21 27.5 mm to (150.5, 82.5)
- moved R8 27.5 mm to (165.7, 47.8)
- moved C11 24.9 mm to (151.3, 36.2)
- moved C12 24.9 mm to (151.1, 58.2)
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Connections:
- C1 pad 1: Sum -> Net-(U1-IN-)
- R6 pad 1: VR4 -> Sum
- R6 pad 2: Sum -> Net-(U1-IN-)
- U1 pad 2: Sum -> Net-(U1-IN-)
Routing:
- net S_out: track 204.1 -> 0.00 mm, vias 1 -> 0
- net VR4: track 183.0 -> 8.67 mm, vias 2 -> 0
- net Net-(U1-IN-): track 0.00 -> 98.8 mm, vias 0 -> 1
- net VR1: track 156.3 -> 65.5 mm, vias 0 -> 1
- net -15V: track 570.4 -> 490.3 mm, vias 1 -> 0
- net X_out: track 225.3 -> 152.9 mm
- net V: track 277.5 -> 208.8 mm, vias 2 -> 3
- net Net-(U13-IN+): track 174.8 -> 126.1 mm
- net Sum: track 71.9 -> 25.0 mm
- net V_out: track 177.9 -> 138.0 mm
- net x: track 204.0 -> 166.3 mm, vias 0 -> 3
- net -V: track 173.2 -> 138.6 mm
- net -x: track 96.7 -> 71.4 mm, vias 1 -> 2
- net Net-(U3-IN-): track 58.6 -> 39.8 mm
- net Net-(R10-Pad2): track 0.00 -> 11.6 mm
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Other:
- board size 200.5 x 120.5 mm -> 153.5 x 120.5 mm
